File: keychron-optical-keyboard.kicad_sch (KiCad schematic)
At the start: 223 parts

Commit message: added readme
Parts:
- added RP?: R_PT, Resistor_SMD:R_0805_2012Metric_Pad1.20x1.40mm_HandSolder, symbol MySymbols:R_PT
Connections:
- net 3v3: now also RP?.2
- net at S?.3 (C): now also RP?.1
- net column 1: now reaches S?.3 (C)
- net column 1: now also S?.3 (C), S?.3 (C), S?.3 (C), S?.3 (C)

Commit message: added connection for few columns
Parts:
- added RP?: R_PT, Resistor_SMD:R_0805_2012Metric_Pad1.20x1.40mm_HandSolder, symbol MySymbols:R_PT
Connections:
- net 3v3: now also RP?.2
- net column 1: now also RP?.1, S?.3 (C)
- net column 2: now reaches S?.3 (C)
- net column 2: now also S?.3 (C), S?.3 (C), S?.3 (C), S?.3 (C), S?.3 (C), RP?.1
Changed lines of the file:
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@@
 (kicad_sch (version 20211123) (generator eeschema)
   (paper "A3")
+  (junction (at 34.29 149.86) (diameter 0) (color 0 0 0 0)
+  )
+  (junction (at 46.99 104.14) (diameter 0) (color 0 0 0 0)
+  )
   (junction (at 13.97 104.14) (diameter 0) (color 0 0 0 0)
   )
@@
   (junction (at 17.78 149.86) (diameter 0) (color 0 0 0 0)
   )
+  (junction (at 46.99 127) (diameter 0) (color 0 0 0 0)
+  )
   (junction (at 13.97 58.42) (diameter 0) (color 0 0 0 0)
   )
+  (junction (at 46.99 58.42) (diameter 0) (color 0 0 0 0)
+  )
+  (junction (at 46.99 81.28) (diameter 0) (color 0 0 0 0)
+  )
+  (junction (at 50.8 149.86) (diameter 0) (color 0 0 0 0)
+  )
   (junction (at 13.97 81.28) (diameter 0) (color 0 0 0 0)
   )
   (junction (at 13.97 149.86) (diameter 0) (color 0 0 0 0)
   )
+  (junction (at 46.99 149.86) (diameter 0) (color 0 0 0 0)
+  )
   (junction (at 30.48 127) (diameter 0) (color 0 0 0 0)
   )
+  (junction (at 30.48 149.86) (diameter 0) (color 0 0 0 0)
+  )
   (junction (at 30.48 104.14) (diameter 0) (color 0 0 0 0)
   )
@@
     (stroke (width 0) (type default) (color 0 0 0 0))
   )
+  (wire (pts (xy 46.99 127) (xy 46.99 149.86))
+    (stroke (width 0) (type default) (color 0 0 0 0))
+  )
   (wire (pts (xy 232.41 64.77) (xy 232.41 66.04))
     (stroke (width 0) (type default) (color 0 0 0 0))
@@
     (stroke (width 0) (type default) (color 0 0 0 0))
   )
+  (wire (pts (xy 34.29 149.86) (xy 34.29 152.4))
+    (stroke (width 0) (type default) (color 0 0 0 0))
+  )
+  (wire (pts (xy 50.8 149.86) (xy 50.8 152.4))
+    (stroke (width 0) (type default) (color 0 0 0 0))
+  )
   (wire (pts (xy 199.39 110.49) (xy 199.39 111.76))
     (stroke (width 0) (type default) (color 0 0 0 0))
@@
     (stroke (width 0) (type default) (color 0 0 0 0))
   )
+  (wire (pts (xy 46.99 81.28) (xy 50.8 81.28))
+    (stroke (width 0) (type default) (color 0 0 0 0))
+  )
   (wire (pts (xy 133.35 133.35) (xy 133.35 134.62))
     (stroke (width 0) (type default) (color 0 0 0 0))
@@
     (stroke (width 0) (type default) (color 0 0 0 0))
   )
-  (wire (pts (xy 30.48 127) (xy 30.48 153.67))
+  (wire (pts (xy 30.48 127) (xy 30.48 149.86))
     (stroke (width 0) (type default) (color 0 0 0 0))
   )
@@
     (stroke (width 0) (type default) (color 0 0 0 0))
   )
+  (wire (pts (xy 50.8 127) (xy 46.99 127))
+    (stroke (width 0) (type default) (color 0 0 0 0))
+  )
   (wire (pts (xy 67.31 133.35) (xy 67.31 134.62))
     (stroke (width 0) (type default) (color 0 0 0 0))
@@
     (stroke (width 0) (type default) (color 0 0 0 0))
   )
+  (wire (pts (xy 30.48 149.86) (xy 30.48 153.67))
+    (stroke (width 0) (type default) (color 0 0 0 0))
+  )
   (wire (pts (xy 116.84 87.63) (xy 116.84 88.9))
     (stroke (width 0) (type default) (color 0 0 0 0))
@@
     (stroke (width 0) (type default) (color 0 0 0 0))
   )
+  (wire (pts (xy 46.99 35.56) (xy 50.8 35.56))
+    (stroke (width 0) (type default) (color 0 0 0 0))
+  )
   (wire (pts (xy 232.41 41.91) (xy 232.41 43.18))
     (stroke (width 0) (type default) (color 0 0 0 0))
@@
     (stroke (width 0) (type default) (color 0 0 0 0))
   )
+  (wire (pts (xy 46.99 58.42) (xy 50.8 58.42))
+    (stroke (width 0) (type default) (color 0 0 0 0))
+  )
   (wire (pts (xy 30.48 104.14) (xy 34.29 104.14))
     (stroke (width 0) (type default) (color 0 0 0 0))
@@
     (stroke (width 0) (type default) (color 0 0 0 0))
   )
+  (wire (pts (xy 46.99 149.86) (xy 50.8 149.86))
+    (stroke (width 0) (type default) (color 0 0 0 0))
+  )
   (wire (pts (xy 34.29 99.06) (xy 34.29 104.14))
     (stroke (width 0) (type default) (color 0 0 0 0))
@@
     (stroke (width 0) (type default) (color 0 0 0 0))
   )
+  (wire (pts (xy 46.99 104.14) (xy 46.99 127))
+    (stroke (width 0) (type default) (color 0 0 0 0))
+  )
   (wire (pts (xy 100.33 30.48) (xy 100.33 35.56))
     (stroke (width 0) (type default) (color 0 0 0 0))
@@
     (stroke (width 0) (type default) (color 0 0 0 0))
   )
+  (wire (pts (xy 46.99 35.56) (xy 46.99 58.42))
+    (stroke (width 0) (type default) (color 0 0 0 0))
+  )
   (wire (pts (xy 83.82 110.49) (xy 83.82 111.76))
     (stroke (width 0) (type default) (color 0 0 0 0))
@@
     (stroke (width 0) (type default) (color 0 0 0 0))
   )
+  (wire (pts (xy 46.99 149.86) (xy 46.99 153.67))
+    (stroke (width 0) (type default) (color 0 0 0 0))
+  )
   (wire (pts (xy 17.78 35.56) (xy 13.97 35.56))
     (stroke (width 0) (type default) (color 0 0 0 0))
@@
     (stroke (width 0) (type default) (color 0 0 0 0))
   )
+  (wire (pts (xy 34.29 149.86) (xy 30.48 149.86))
+    (stroke (width 0) (type default) (color 0 0 0 0))
+  )
   (wire (pts (xy 17.78 99.06) (xy 17.78 104.14))
     (stroke (width 0) (type default) (color 0 0 0 0))
@@
     (stroke (width 0) (type default) (color 0 0 0 0))
   )
-  (wire (pts (xy 34.29 144.78) (xy 34.29 152.4))
+  (wire (pts (xy 34.29 144.78) (xy 34.29 149.86))
     (stroke (width 0) (type default) (color 0 0 0 0))
   )
@@
     (stroke (width 0) (type default) (color 0 0 0 0))
   )
+  (wire (pts (xy 46.99 104.14) (xy 50.8 104.14))
+    (stroke (width 0) (type default) (color 0 0 0 0))
+  )
   (wire (pts (xy 17.78 152.4) (xy 17.78 149.86))
     (stroke (width 0) (type default) (color 0 0 0 0))
@@
     (stroke (width 0) (type default) (color 0 0 0 0))
   )
+  (wire (pts (xy 46.99 58.42) (xy 46.99 81.28))
+    (stroke (width 0) (type default) (color 0 0 0 0))
+  )
+  (wire (pts (xy 46.99 81.28) (xy 46.99 104.14))
+    (stroke (width 0) (type default) (color 0 0 0 0))
+  )
   (wire (pts (xy 298.45 41.91) (xy 298.45 43.18))
     (stroke (width 0) (type default) (color 0 0 0 0))
   )
+  (global_label "3v3" (shape output) (at 50.8 160.02 270) (fields_autoplaced)
+    (effects (font (size 1 1)) (justify right))
+    (property "Intersheet References" "${INTERSHEET_REFS}" (id 0) (at 50.8625 164.5867 90)
+      (effects (font (size 1 1)) (justify right) hide)
+    )
+  )
   (global_label "column 1" (shape input) (at 30.48 153.67 270) (fields_autoplaced)
     (effects (font (size 1.27 1.27)) (justify right))
@@
     )
   )
+  (global_label "column 2" (shape input) (at 46.99 153.67 270) (fields_autoplaced)
+    (effects (font (size 1.27 1.27)) (justify right))
+    (property "Intersheet References" "${INTERSHEET_REFS}" (id 0) (at 46.9106 165.1545 90)
+      (effects (font (size 1.27 1.27)) (justify right) hide)
+    )
+  )
   (global_label "column 0" (shape input) (at 13.97 153.67 270) (fields_autoplaced)
     (effects (font (size 1.27 1.27)) (justify right))
@@
     (pin "4")
   )
+  (symbol (lib_id "MySymbols:R_PT") (at 50.8 156.21 0) (unit 1)
+    (in_bom yes) (on_board yes) (fields_autoplaced)
+    (property "Reference" "RP?" (id 0) (at 52.832 156.21 90))
+    (property "Value" "R_PT" (id 1) (at 50.8 156.21 90))
+    (property "Footprint" "Resistor_SMD:R_0805_2012Metric_Pad1.20x1.40mm_HandSolder" (id 2) (at 49.022 156.21 90)
+      (effects (font (size 1.27 1.27)) hide)
+    )
+    (property "Datasheet" "~" (id 3) (at 50.8 156.21 0)
+      (effects (font (size 1.27 1.27)) hide)
+    )
+    (property "JLC" "0805-2012" (id 4) (at 57.15 152.4 0)
+      (effects (font (size 1.27 1.27)) hide)
+    )
+    (property "LCSC" "C17713" (id 5) (at 57.15 154.94 0)
+      (effects (font (size 1.27 1.27)) hide)
+    )
+    (pin "1")
+    (pin "2")
+  )
   (symbol (lib_id "power:GND") (at 190.5 29.21 0) (unit 1)
     (in_bom yes) (on_board yes) (fields_autoplaced)
@@
       (reference "RP?") (unit 1) (value "R_PT") (footprint "Resistor_SMD:R_0805_2012Metric_Pad1.20x1.40mm_HandSolder")
     )
+    (path "/610e755d-52f4-48f2-b762-bdaf664a5c4a"
+      (reference "RP?") (unit 1) (value "R_PT") (footprint "Resistor_SMD:R_0805_2012Metric_Pad1.20x1.40mm_HandSolder")
+    )

Commit message: added a switch
Parts:
- added S?: OptSw, MyFootprints:Keychron_Optical_Switch_1u, symbol MySymbols:OptSw
Connections:
- net GND: now also S?.2 (IR_K), S?.4 (E)
Changed lines of the file:
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@@
     (stroke (width 0) (type default) (color 0 0 0 0))
   )
+  (wire (pts (xy 298.45 87.63) (xy 298.45 88.9))
+    (stroke (width 0) (type default) (color 0 0 0 0))
+  )
   (wire (pts (xy 116.84 30.48) (xy 116.84 35.56))
     (stroke (width 0) (type default) (color 0 0 0 0))
@@
     (stroke (width 0) (type default) (color 0 0 0 0))
   )
+  (wire (pts (xy 298.45 99.06) (xy 298.45 104.14))
+    (stroke (width 0) (type default) (color 0 0 0 0))
+  )
   (wire (pts (xy 298.45 64.77) (xy 298.45 66.04))
     (stroke (width 0) (type default) (color 0 0 0 0))
@@
     (pin "2")
   )
+  (symbol (lib_id "MySymbols:OptSw") (at 298.45 93.98 0) (unit 1)
+    (in_bom yes) (on_board yes) (fields_autoplaced)
+    (property "Reference" "S?" (id 0) (at 302.26 101.6 0)
+      (effects (font (size 1.27 1.27)) (justify left))
+    )
+    (property "Value" "OptSw" (id 1) (at 299.72 104.14 0)
+      (effects (font (size 1 1)) (justify left))
+    )
+    (property "Footprint" "MyFootprints:Keychron_Optical_Switch_1u" (id 2) (at 295.91 96.52 0)
+      (effects (font (size 1.27 1.27)) hide)
+    )
+    (property "Datasheet" "~" (id 3) (at 300.99 93.98 0)
+      (effects (font (size 1.27 1.27)) hide)
+    )
+    (pin "1")
+    (pin "2")
+    (pin "3")
+    (pin "4")
+  )
   (symbol (lib_id "power:GND") (at 273.05 120.65 0) (unit 1)
     (in_bom yes) (on_board yes) (fields_autoplaced)
@@
     (pin "1")
   )
+  (symbol (lib_id "power:GND") (at 306.07 97.79 0) (unit 1)
+    (in_bom yes) (on_board yes) (fields_autoplaced)
+    (property "Reference" "#PWR?" (id 0) (at 306.07 104.14 0)
+      (effects (font (size 1.27 1.27)) hide)
+    )
+    (property "Value" "GND" (id 1) (at 306.07 101.6 0))
+    (property "Footprint" "" (id 2) (at 306.07 97.79 0)
+      (effects (font (size 1.27 1.27)) hide)
+    )
+    (property "Datasheet" "" (id 3) (at 306.07 97.79 0)
+      (effects (font (size 1.27 1.27)) hide)
+    )
+    (pin "1")
+  )
   (symbol (lib_id "MySymbols:OptSw") (at 100.33 25.4 0) (unit 1)
     (in_bom yes) (on_board yes) (fields_autoplaced)
@@
     (pin "4")
   )
+  (symbol (lib_id "power:GND") (at 298.45 87.63 180) (unit 1)
+    (in_bom yes) (on_board yes) (fields_autoplaced)
+    (property "Reference" "#PWR?" (id 0) (at 298.45 81.28 0)
+      (effects (font (size 1.27 1.27)) hide)
+    )
+    (property "Value" "GND" (id 1) (at 298.45 83.82 0))
+    (property "Footprint" "" (id 2) (at 298.45 87.63 0)
+      (effects (font (size 1.27 1.27)) hide)
+    )
+    (property "Datasheet" "" (id 3) (at 298.45 87.63 0)
+      (effects (font (size 1.27 1.27)) hide)
+    )
+    (pin "1")
+  )
   (symbol (lib_id "MySymbols:R_IR") (at 372.11 63.5 0) (unit 1)
     (in_bom yes) (on_board yes) (fields_autoplaced)
@@
       (reference "#PWR0322") (unit 1) (value "GND") (footprint "")
     )
+    (path "/88ec5fa8-198f-4375-a657-e37a0fa71051"
+      (reference "#PWR?") (unit 1) (value "GND") (footprint "")
+    )
+    (path "/cd89deb9-2fdf-4837-993e-173522465931"
+      (reference "#PWR?") (unit 1) (value "GND") (footprint "")
+    )
     (path "/01ffcdf4-f858-488e-bd1c-e2ed146f4dae"
       (reference "RL?") (unit 1) (value "R_IR") (footprint "Resistor_SMD:R_0805_2012Metric_Pad1.20x1.40mm_HandSolder")
@@
       (reference "S?") (unit 1) (value "OptSw") (footprint "MyFootprints:Keychron_Optical_Switch_1u")
     )
+    (path "/0f3f2d65-5fa7-49ef-a1a5-d0252bcda31c"
+      (reference "S?") (unit 1) (value "OptSw") (footprint "MyFootprints:Keychron_Optical_Switch_1u")
+    )

Commit message: connected all columns and rows
Parts:
- added RP? (x20): R_PT, Resistor_SMD:R_0805_2012Metric_Pad1.20x1.40mm_HandSolder, symbol MySymbols:R_PT
Connections:
- net 3v3: now also RP?.2, RP?.2, RP?.2, RP?.2, RP?.2, RP?.2, RP?.2, RP?.2, RP?.2, RP?.2, RP?.2, RP?.2, RP?.2, RP?.2, RP?.2, RP?.2, RP?.2, RP?.2, RP?.2, RP?.2
- net column 12: now reaches S?.3 (C)
- net column 12: now also RL?.1, RL?.1, RL?.1, RL?.1, RL?.1, RL?.1, RL?.1, RL?.1, RL?.1, RL?.1, RL?.1, RL?.1, RL?.1, S?.3 (C), S?.3 (C), S?.3 (C), S?.3 (C), S?.3 (C), RP?.1
- net column 13: now reaches S?.3 (C)
- net column 13: now also S?.3 (C), S?.3 (C), S?.3 (C), S?.3 (C), RP?.1
- net row 1: now reaches RL?.1
- net row 1: now also RL?.1, RL?.1, RL?.1, RL?.1, RL?.1, RL?.1, RL?.1, RL?.1, RL?.1, RL?.1, RL?.1, RL?.1, RL?.1, RL?.1, RL?.1, RL?.1, RL?.1, RL?.1, RL?.1, RL?.1, RL?.1, RL?.1
- net column 17: now reaches RL?.1
- net column 17: now also RL?.1, RL?.1, RL?.1, RL?.1, RL?.1, RL?.1, RL?.1, RL?.1, RL?.1, RL?.1, RL?.1, RL?.1, RL?.1, RL?.1, RL?.1, RL?.1, RL?.1, RL?.1, S?.3 (C), S?.3 (C), S?.3 (C), S?.3 (C), RP?.1
- net column 11: now reaches S?.3 (C)
- net column 11: now also S?.3 (C), S?.3 (C), S?.3 (C), S?.3 (C), S?.3 (C), RP?.1
- net column 7: now reaches S?.3 (C)
- net column 7: now also RL?.1, RL?.1, RL?.1, RL?.1, RL?.1, RL?.1, RL?.1, RL?.1, RL?.1, RL?.1, RL?.1, RL?.1, RL?.1, RL?.1, RL?.1, RL?.1, RL?.1, S?.3 (C), S?.3 (C), S?.3 (C), S?.3 (C), S?.3 (C), RP?.1
- net row 2: now reaches RL?.1
- net row 2: now also RL?.1, RL?.1, RL?.1, RL?.1, RL?.1, RL?.1, RL?.1, RL?.1, RL?.1, RL?.1, RL?.1, RL?.1, RL?.1, RL?.1, RL?.1, RL?.1, RL?.1, RL?.1, RL?.1, RL?.1, RL?.1, RL?.1
- net column 4: now reaches S?.3 (C)
- net column 4: now also S?.3 (C), S?.3 (C), S?.3 (C), S?.3 (C), S?.3 (C), RP?.1
- net column 20: now reaches S?.3 (C)
- net column 20: now also S?.3 (C), RP?.1
- net column 3: now reaches S?.3 (C)
- net column 3: now also S?.3 (C), S?.3 (C), S?.3 (C), S?.3 (C), S?.3 (C), RP?.1
- net row 0: now reaches RL?.1
- net row 0: now also RL?.1, RL?.1, RL?.1, RL?.1, RL?.1, RL?.1, RL?.1, RL?.1, RL?.1, RL?.1, RL?.1, RL?.1, RL?.1, RL?.1, RL?.1
- net column 16: now reaches S?.3 (C)
- net column 16: now also S?.3 (C), S?.3 (C), S?.3 (C), RP?.1
- net column 8: now reaches S?.3 (C)
- net column 8: now also S?.3 (C), S?.3 (C), S?.3 (C), S?.3 (C), S?.3 (C), RP?.1
- net column 6: now reaches S?.3 (C)
- net column 6: now also S?.3 (C), S?.3 (C), S?.3 (C), S?.3 (C), S?.3 (C), RP?.1
- net column 22: now reaches S?.3 (C)
- net column 22: now also S?.3 (C), RP?.1
- net column 9: now reaches S?.3 (C)
- net column 9: now also S?.3 (C), S?.3 (C), S?.3 (C), S?.3 (C), S?.3 (C), RP?.1
- net column 5: now reaches S?.3 (C)
- net column 5: now also S?.3 (C), S?.3 (C), S?.3 (C), S?.3 (C), S?.3 (C), RP?.1
- net column 19: now reaches S?.3 (C)
- net column 19: now also S?.3 (C), RP?.1
- net column 10: now reaches S?.3 (C)
- net column 10: now also S?.3 (C), S?.3 (C), S?.3 (C), S?.3 (C), S?.3 (C), RP?.1
- net column 15: now reaches S?.3 (C)
- net column 15: now also S?.3 (C), S?.3 (C), S?.3 (C), S?.3 (C), RP?.1
- net column 14: now reaches S?.3 (C)
- net column 14: now also S?.3 (C), S?.3 (C), S?.3 (C), S?.3 (C), RP?.1
- net column 21: now reaches S?.3 (C)
- net column 21: now also S?.3 (C), RP?.1
- net column 18: now reaches S?.3 (C)
- net column 18: now also S?.3 (C), S?.3 (C), RP?.1
