File: keychron-optical-keyboard.kicad_sch (KiCad schematic)
At the start: 246 parts

Commit message: picking better componenets, starting to connect schema
Parts:
- added U1: STM32F303ZETx, Package_QFP:LQFP-144_20x20mm_P0.5mm, symbol MCU_ST_STM32F3:STM32F303ZETx
- added U2: LP5030, Package_DFN_QFN:VQFN-46-1EP_5x6mm_P0.4mm_EP2.8x3.8mm, symbol Driver_LED:LP5036
Connections:
- net column 0: now also U1.68 (PE15)
- net column 1: now also U1.67 (PE14)
- net column 10: now also U1.4 (PE5)
- net column 11: now also U1.3 (PE4)
- net column 12: now also U1.12 (PF2), U1.2 (PE3)
- net column 13: now also U1.1 (PE2)
- net column 14: now also U1.142 (PE1)
- net column 15: now also U1.141 (PE0)
- net column 16: now also U1.55 (PF15)
- net column 17: now also U1.13 (PF3), U1.54 (PF14)
- net column 18: now also U1.53 (PF13)
- net column 19: now also U1.50 (PF12)
- net column 2: now also U1.66 (PE13)
- net column 20: now also U1.49 (PF11)
- net column 21: now also U1.22 (PF10)
- net column 22: now also U1.21 (PF9)
- net column 3: now also U1.65 (PE12)
- net column 4: now also U1.64 (PE11)
- net column 5: now also U1.63 (PE10)
- net column 6: now also U1.60 (PE9)
- net column 7: now also U1.14 (PF4), U1.59 (PE8)
- net column 8: now also U1.58 (PE7)
- net column 9: now also U1.5 (PE6)
- net row 0: now also U1.19 (PF7)
- net row 1: now also U1.18 (PF6)
- net row 2: now also U1.15 (PF5)
- new net: U2.37 (GND), U2.46 (GND), U2.47 (GND)
- new net: U1.107 (VSS), U1.120 (VSS), U1.130 (VSS), U1.143 (VSS), U1.16 (VSS), U1.38 (VSS), U1.51 (VSS), U1.61 (VSS), U1.71 (VSS), U1.83 (VSS), U1.94 (VSS)
- new net column 23: U1.20 (PF8)
